Commit message: Fix RG body mounts and prepare ROS suite 1.3.1 (#10)
Declare the RG2 and RG6 body connections as fixed in simplified descriptions
and plain URDFs, matching the detailed descriptions. MoveIt no longer needs an
unavailable body-joint measurement. The default mounting pose is unchanged.

Update package versions and release notes for this fix and the separately
merged launch fix from PR #7 and Gazebo resource fix contributed in PR #6.

Fixes #5

File: onrobot_rg2/urdf/onrobot_rg2.urdf (robot description, URDF)
Before this commit: robot onrobot_rg2, 14 links, 13 joints
Joints:
- joint body_joint: axis 0 0 -1 -> (none); limit lower=-1.57079632679 upper=1.57079632679 effort=0 velocity=0 -> (none); type revolute -> fixed

File: onrobot_rg2/urdf/onrobot_rg2_macro.xacro (robot description, xacro)
@@ -275,5 +275,5 @@
         </collision>
       </link>
-      <joint name="${prefix}body_joint" type="revolute">
+      <joint name="${prefix}body_joint" type="fixed">
         <origin
           xyz="0 0 0.04734"
@@ -281,10 +281,4 @@
         <parent link="${prefix}base_link"/>
         <child link="${prefix}body_link"/>
-        <axis xyz="0 0 1"/>
-        <limit
-          lower="-1.5708"
-          upper="1.5708"
-          effort="0"
-          velocity="0"/>
       </joint>
       <!-- ============================================================= -->

File: onrobot_rg6/urdf/onrobot_rg6.urdf (robot description, URDF)
Before this commit: robot onrobot_rg6, 12 links, 11 joints
Joints:
- joint body_joint: axis 0 0 1 -> (none); limit lower=-1.5708 upper=1.5708 effort=140 velocity=1 -> (none); type revolute -> fixed

File: onrobot_rg6/urdf/onrobot_rg6_macro.xacro (robot description, xacro)
@@ -261,5 +261,5 @@
         </collision>
       </link>
-      <joint name="${prefix}body_joint" type="revolute">
+      <joint name="${prefix}body_joint" type="fixed">
         <origin
           xyz="0 0 0.0503000000000003"
@@ -267,10 +267,4 @@
         <parent link="${prefix}base_link"/>
         <child link="${prefix}body_link"/>
-        <axis xyz="0 0 1"/>
-        <limit
-          lower="-1.5708"
-          upper="1.5708"
-          effort="0"
-          velocity="0"/>
       </joint>
       <!-- ================= Right outer proximal finger ================= -->
