Commit message: Add grip_stroke declarations to RG xacro macros

File: onrobot_rg2/urdf/onrobot_rg2_macro.xacro (robot description, xacro)
@@ -777,4 +777,11 @@
         <mu2>0.4</mu2>
       </gazebo>
+      <!-- Semantic aperture joint. The visual finger-angle mapping is intentionally
+      not claimed until calibrated; this joint is the ROS command/state API. -->
+      <link name="${prefix}grip_stroke_control_link"/>
+      <joint name="${prefix}grip_stroke" type="prismatic">
+        <parent link="${prefix}base_link"/><child link="${prefix}grip_stroke_control_link"/>
+        <axis xyz="1 0 0"/><limit lower="0" upper="0.110" effort="40" velocity="1"/>
+      </joint>
   </xacro:macro>
 </robot>

File: onrobot_rg6/urdf/onrobot_rg6_macro.xacro (robot description, xacro)
@@ -680,4 +680,11 @@
         <mu2>0.4</mu2>
       </gazebo>
+      <!-- Semantic aperture control joint; visual finger-angle calibration remains
+      a separate requirement and is not silently approximated here. -->
+      <link name="${prefix}grip_stroke_control_link"/>
+      <joint name="${prefix}grip_stroke" type="prismatic">
+        <parent link="${prefix}base_link"/><child link="${prefix}grip_stroke_control_link"/>
+        <axis xyz="1 0 0"/><limit lower="0" upper="0.160" effort="120" velocity="1"/>
+      </joint>
   </xacro:macro>
 </robot>
